File: src/PCB_KICAD/EpromWriter/EpromWriter.kicad_pcb (KiCad board)
At the start: 2 copper layers, 5 parts, among them U1 74LS367, U2 74LS367, U3 MC34063AP

Commit message: Menü hozzáadása és néhány apróbb változtatás
Parts:
- added C2: 100n, Capacitor_THT:C_Disc_D3.0mm_W2.0mm_P2.50mm, F.Cu at (114.5, 84.3)
- added C3: 1n, Capacitor_THT:C_Disc_D3.0mm_W1.6mm_P2.50mm, F.Cu at (129.9, 81.9)
- added C4: 100n, Capacitor_THT:C_Disc_D3.0mm_W2.0mm_P2.50mm, F.Cu at (114.5, 87.8)
- added C5: 3.3u, Capacitor_THT:C_Radial_D6.3mm_H5.0mm_P2.50mm, F.Cu at (140.2, 24.9)
- added C6: 47u/35v, Capacitor_THT:CP_Radial_D5.0mm_P2.00mm, F.Cu at (137.1, 66.5)
- added C7: 33u, Capacitor_THT:C_Radial_D6.3mm_H5.0mm_P2.50mm, F.Cu at (115.6, 75.0)
- added D1: 1N4001, Diode_THT:D_DO-41_SOD81_P10.16mm_Horizontal, F.Cu at (142.1, 36.7)
- added D2: 1N4148, Diode_THT:D_DO-35_SOD27_P7.62mm_Horizontal, F.Cu at (146.8, 44.3)
- added D3: 1N4148, Diode_THT:D_DO-35_SOD27_P7.62mm_Horizontal, F.Cu at (115.6, 40.0)
- added D5: 1N4001, Diode_THT:D_DO-41_SOD81_P10.16mm_Horizontal, F.Cu at (138.7, 48.4)
- added D6: RED, LED_THT:LED_D5.0mm, F.Cu at (123.3, 84.1)
- added J1: Barrel_Jack, Connector_BarrelJack:BarrelJack_Kycon_KLDX-0202-xC_Horizontal, F.Cu at (116.8, 35.2)
- added J3: Conn_01x04_Pin, Connector_JST:JST_EH_B4B-EH-A_1x04_P2.50mm_Vertical, F.Cu at (98.5, 23.0)
- added J4: Conn_01x03_Pin, Connector_JST:JST_EH_B3B-EH-A_1x03_P2.50mm_Vertical, F.Cu at (86.5, 23.1)
- added JP1: Jumper_3_Bridged12, Connector_JST:JST_EH_B3B-EH-A_1x03_P2.50mm_Vertical, F.Cu at (147.9, 30.6)
- added JP2: Jumper_3_Bridged12, Connector_JST:JST_EH_B3B-EH-A_1x03_P2.50mm_Vertical, F.Cu at (154.4, 54.1)
- added L1: 100uH, Capacitor_THT:CP_Radial_D5.0mm_P2.50mm, F.Cu at (136.8, 73.1)
- added R4: 220, Resistor_THT:R_Axial_DIN0207_L6.3mm_D2.5mm_P15.24mm_Horizontal, F.Cu at (136.3, 78.4)
- added R5: 0.33/10W, Resistor_THT:R_Radial_Power_L11.0mm_W7.0mm_P5.00mm, F.Cu at (131.3, 45.4)
- added R7: 1.2k, Resistor_THT:R_Axial_DIN0207_L6.3mm_D2.5mm_P7.62mm_Horizontal, F.Cu at (142.9, 72.4)
- added U4: LM7805_TO220, Package_TO_SOT_THT:TO-220-3_Vertical, F.Cu at (153.3, 40.9)
- added U5: ESP32_NODEMCU, AndrewLib:MODULE_ESP32_NODEMCU, F.Cu at (67.3, 48.5)
- C1: value 1n -> 100n; footprint Capacitor_THT:C_Disc_D3.0mm_W1.6mm_P2.50mm -> Capacitor_THT:C_Disc_D3.0mm_W2.0mm_P2.50mm
- moved U2 46.7 mm to (126.8, 97.8)
- moved RN1 46.0 mm to (125.7, 93.6), turned to 0 degrees
- moved U3 34.5 mm to (127.7, 22.4)
- moved C1 14.4 mm to (114.5, 80.7)
- moved U1 14.0 mm to (90.9, 42.3)
Connections:
- C1 pad 1: GNDREF -> VCC
- C1 pad 2: Net-(U3-TC) -> GNDREF
- U3 pad 1: GNDREF -> Net-(D4-A)
- U3 pad 4: unconnected-(U3-GND-Pad4) -> GNDREF
- U3 pad 5: unconnected-(U3-Vfb-Pad5) -> Net-(U3-Vfb)
- U3 pad 7: unconnected-(U3-Ipk-Pad7) -> Net-(U3-Ipk)
- U3 pad 8: unconnected-(U3-DC-Pad8) -> Net-(U3-DC)
Routing:
- net GNDREF: track 44.1 -> 153.9 mm
- net /MCU/encButton: track 0.00 -> 58.0 mm
- net /MCU/encB: track 0.00 -> 50.0 mm
- net Net-(D2-K): track 0.00 -> 43.3 mm
- net /MCU/encA: track 0.00 -> 40.6 mm
- net Net-(D5-A): track 0.00 -> 32.0 mm
- net /MCU/SDA: track 0.00 -> 24.6 mm
- net /MCU/SCL: track 0.00 -> 24.0 mm
- net Net-(D2-A): track 0.00 -> 21.7 mm
- net /DO3: track 21.0 -> 0.00 mm
- net +12V: track 0.00 -> 18.4 mm
- net VCC: track 44.6 -> 60.9 mm
- net +5V: track 13.0 -> 0.00 mm
- net Net-(D1-K): track 0.00 -> 12.9 mm
- net /DO2: track 7.55 -> 0.00 mm
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