File: src/PCB_KICAD/EpromWriter/EpromWriter.kicad_sch (KiCad schematic)
At the start: 3 parts, among them U1 74LS367, U2 74LS367

Commit message: Menü hozzáadása és néhány apróbb változtatás
Other:
- sheet Untitled Sheet renamed PSU for Eprom Writer
- added sheet Jumpers (Jumpers.kicad_sch)
- added sheet MCU (mcu.kicad_sch)
- sheet PSU for Eprom Writer: file untitled.kicad_sch -> PSU_for_Writer.kicad_sch
Changed lines of the file:
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@@
 (kicad_sch (version 20230121) (generator eeschema)
   (paper "A4")
+  (title_block
+    (date "2023-08-13")
+    (rev "1.1")
+  )
   (junction (at 60.96 43.18) (diameter 0) (color 0 0 0 0)
   )
@@
   (symbol (lib_id "power:GNDREF") (at 80.01 71.12 0) (unit 1)
     (in_bom yes) (on_board yes) (dnp no) (fields_autoplaced)
-    (property "Reference" "#PWR06" (at 80.01 77.47 0)
+    (property "Reference" "#PWR02" (at 80.01 77.47 0)
       (effects (font (size 1.27 1.27)) hide)
     )
@@
       (project "EpromWriter"
         (path "/01f26431-3776-438d-a17f-fa62f387fe06"
-          (reference "#PWR06") (unit 1)
+          (reference "#PWR02") (unit 1)
         )
       )
@@
   (symbol (lib_id "power:VCC") (at 20.32 29.21 0) (unit 1)
     (in_bom yes) (on_board yes) (dnp no) (fields_autoplaced)
-    (property "Reference" "#PWR03" (at 20.32 33.02 0)
+    (property "Reference" "#PWR01" (at 20.32 33.02 0)
       (effects (font (size 1.27 1.27)) hide)
     )
@@
       (project "EpromWriter"
         (path "/01f26431-3776-438d-a17f-fa62f387fe06"
-          (reference "#PWR03") (unit 1)
+          (reference "#PWR01") (unit 1)
         )
       )
@@
   (symbol (lib_id "power:GNDREF") (at 80.01 120.65 0) (unit 1)
     (in_bom yes) (on_board yes) (dnp no) (fields_autoplaced)
-    (property "Reference" "#PWR07" (at 80.01 127 0)
+    (property "Reference" "#PWR03" (at 80.01 127 0)
       (effects (font (size 1.27 1.27)) hide)
     )
@@
       (project "EpromWriter"
         (path "/01f26431-3776-438d-a17f-fa62f387fe06"
-          (reference "#PWR07") (unit 1)
+          (reference "#PWR03") (unit 1)
         )
       )
@@
     )
   )
-  (sheet (at -66.04 48.26) (size 52.07 53.34) (fields_autoplaced)
+  (sheet (at -39.37 88.9) (size 21.59 12.7) (fields_autoplaced)
     (stroke (width 0.1524) (type solid))
     (fill (color 0 0 0 0.0000))
-    (property "Sheetname" "Untitled Sheet" (at -66.04 47.5484 0)
+    (property "Sheetname" "Jumpers" (at -39.37 88.1884 0)
       (effects (font (size 1.27 1.27)) (justify left bottom))
     )
-    (property "Sheetfile" "untitled.kicad_sch" (at -66.04 102.1846 0)
+    (property "Sheetfile" "Jumpers.kicad_sch" (at -39.37 102.1846 0)
       (effects (font (size 1.27 1.27)) (justify left top))
     )
     (instances
       (project "EpromWriter"
+        (path "/01f26431-3776-438d-a17f-fa62f387fe06" (page "3"))
+      )
+    )
+  )
+  (sheet (at -66.04 48.26) (size 22.86 13.97) (fields_autoplaced)
+    (stroke (width 0.1524) (type solid))
+    (fill (color 0 0 0 0.0000))
+    (property "Sheetname" "PSU for Eprom Writer" (at -66.04 47.5484 0)
+      (effects (font (size 1.27 1.27)) (justify left bottom))
+    )
+    (property "Sheetfile" "PSU_for_Writer.kicad_sch" (at -66.04 62.8146 0)
+      (effects (font (size 1.27 1.27)) (justify left top))
+    )
+    (instances
+      (project "EpromWriter"
         (path "/01f26431-3776-438d-a17f-fa62f387fe06" (page "2"))
       )
     )
+  )
+  (sheet (at -33.02 48.26) (size 17.78 13.97) (fields_autoplaced)
+    (stroke (width 0.1524) (type solid))
+    (fill (color 0 0 0 0.0000))
+    (property "Sheetname" "MCU" (at -33.02 47.5484 0)
+      (effects (font (size 1.27 1.27)) (justify left bottom))
+    )
+    (property "Sheetfile" "mcu.kicad_sch" (at -33.02 62.8146 0)
+      (effects (font (size 1.27 1.27)) (justify left top))
+    )
+    (instances
+      (project "EpromWriter"
+        (path "/01f26431-3776-438d-a17f-fa62f387fe06" (page "4"))
+      )
+    )
